Commit message: 两轮驱动车第一版修改

File: src/turtlebot3/turtlebot3_description/urdf/turtlebot3_burger.urdf.xacro (robot description, xacro)
@@ -116,5 +116,5 @@
     <parent link="base_link"/>
     <child link="base_scan"/>
-    <origin xyz="-0.032 0 0.172" rpy="0 0 0"/>
+    <origin xyz="0.0 0 0.07" rpy="0 0 0"/>
   </joint>
   <link name="base_scan">

File: src/turtlebot3/turtlebot3_description/urdf/turtlebot3_burger_for_autorace.urdf.xacro (robot description, xacro)
@@ -116,5 +116,5 @@
     <parent link="base_link"/>
     <child link="base_scan"/>
-    <origin xyz="-0.032 0 0.172" rpy="0 0 0"/>
+    <origin xyz="0.0 0 0.07" rpy="0 0 0"/>
   </joint>
   <link name="base_scan">

File: src/turtlebot3/turtlebot3_description/urdf/turtlebot3_burger_for_autorace_2020.urdf.xacro (robot description, xacro)
@@ -116,5 +116,5 @@
     <parent link="base_link"/>
     <child link="base_scan"/>
-    <origin xyz="-0.032 0 0.172" rpy="0 0 0"/>
+    <origin xyz="0.0 0 0.07" rpy="0 0 0"/>
   </joint>
   <link name="base_scan">
