Commit message: 四轮驱动第一版

File: src/turtlebot3/turtlebot3_description/urdf_next/turtlebot3_moguarder.gazebo.xacro (robot description, xacro)
@@ -78,6 +78,6 @@
     <material>Gazebo/Grey</material>
   </gazebo>
-  <gazebo reference="wheel_left_link">
-    <mu1>0.35</mu1>
+  <gazebo reference="wheel_left_front_link">
+    <mu1>0.75</mu1>
     <mu2>0.35</mu2>
     <kp>500000.0</kp>
@@ -88,6 +88,6 @@
     <material>Gazebo/FlatBlack</material>
   </gazebo>
-  <gazebo reference="wheel_right_link">
-    <mu1>0.35</mu1>
+  <gazebo reference="wheel_right_front_link">
+    <mu1>0.75</mu1>
     <mu2>0.35</mu2>
     <kp>500000.0</kp>
@@ -98,11 +98,22 @@
     <material>Gazebo/FlatBlack</material>
   </gazebo>
-  <gazebo reference="caster_back_link">
-    <mu1>0.08</mu1>
-    <mu2>0.08</mu2>
-    <kp>1000000.0</kp>
-    <kd>100.0</kd>
-    <minDepth>0.001</minDepth>
-    <maxVel>1.0</maxVel>
+  <gazebo reference="wheel_left_rear_link">
+    <mu1>0.85</mu1>
+    <mu2>0.40</mu2>
+    <kp>500000.0</kp>
+    <kd>10.0</kd>
+    <minDepth>0.001</minDepth>
+    <maxVel>0.1</maxVel>
+    <fdir1>1 0 0</fdir1>
+    <material>Gazebo/FlatBlack</material>
+  </gazebo>
+  <gazebo reference="wheel_right_rear_link">
+    <mu1>0.85</mu1>
+    <mu2>0.40</mu2>
+    <kp>500000.0</kp>
+    <kd>10.0</kd>
+    <minDepth>0.001</minDepth>
+    <maxVel>0.1</maxVel>
+    <fdir1>1 0 0</fdir1>
     <material>Gazebo/FlatBlack</material>
   </gazebo>
@@ -115,22 +126,20 @@
   </gazebo>
   <gazebo>
-    <plugin name="moguarder_controller" filename="libgazebo_ros_diff_drive.so">
+    <plugin name="moguarder_skid_steer_controller" filename="libgazebo_ros_skid_steer_drive.so">
       <commandTopic>cmd_vel</commandTopic>
       <odometryTopic>odom</odometryTopic>
       <odometryFrame>odom</odometryFrame>
-      <odometrySource>world</odometrySource>
-      <publishOdomTF>true</publishOdomTF>
       <robotBaseFrame>base_footprint</robotBaseFrame>
+      <updateRate>50</updateRate>
+      <leftFrontJoint>wheel_left_front_joint</leftFrontJoint>
+      <rightFrontJoint>wheel_right_front_joint</rightFrontJoint>
+      <leftRearJoint>wheel_left_rear_joint</leftRearJoint>
+      <rightRearJoint>wheel_right_rear_joint</rightRearJoint>
+      <wheelSeparation>0.156</wheelSeparation>
+      <wheelDiameter>0.066</wheelDiameter>
+      <torque>12</torque>
+      <broadcastTF>true</broadcastTF>
       <publishWheelTF>false</publishWheelTF>
-      <publishTf>true</publishTf>
       <publishWheelJointState>true</publishWheelJointState>
-      <legacyMode>false</legacyMode>
-      <updateRate>50</updateRate>
-      <leftJoint>wheel_left_joint</leftJoint>
-      <rightJoint>wheel_right_joint</rightJoint>
-      <wheelSeparation>0.150</wheelSeparation>
-      <wheelDiameter>0.066</wheelDiameter>
-      <wheelAcceleration>1.5</wheelAcceleration>
-      <wheelTorque>12</wheelTorque>
       <rosDebugLevel>na</rosDebugLevel>
     </plugin>

File: src/turtlebot3/turtlebot3_description/urdf_next/turtlebot3_moguarder.urdf.xacro (robot description, xacro)
@@ -702,11 +702,11 @@
     </inertial>
   </link>
-  <joint name="wheel_left_joint" type="continuous">
-    <parent link="base_link"/>
-    <child link="wheel_left_link"/>
-    <origin xyz="0.0 0.075 0.023" rpy="-1.57 0 0"/>
+  <joint name="wheel_left_front_joint" type="continuous">
+    <parent link="base_link"/>
+    <child link="wheel_left_front_link"/>
+    <origin xyz="0.060 0.078 0.023" rpy="-1.57 0 0"/>
     <axis xyz="0 0 1"/>
   </joint>
-  <link name="wheel_left_link">
+  <link name="wheel_left_front_link">
     <visual>
       <origin xyz="0 0 0" rpy="1.57 0 0"/>
@@ -730,11 +730,11 @@
     </inertial>
   </link>
-  <joint name="wheel_right_joint" type="continuous">
-    <parent link="base_link"/>
-    <child link="wheel_right_link"/>
-    <origin xyz="0.0 -0.075 0.023" rpy="-1.57 0 0"/>
+  <joint name="wheel_right_front_joint" type="continuous">
+    <parent link="base_link"/>
+    <child link="wheel_right_front_link"/>
+    <origin xyz="0.060 -0.078 0.023" rpy="-1.57 0 0"/>
     <axis xyz="0 0 1"/>
   </joint>
-  <link name="wheel_right_link">
+  <link name="wheel_right_front_link">
     <visual>
       <origin xyz="0 0 0" rpy="1.57 0 0"/>
@@ -758,19 +758,88 @@
     </inertial>
   </link>
-  <joint name="caster_back_joint" type="fixed">
-    <parent link="base_link"/>
-    <child link="caster_back_link"/>
-    <origin xyz="-0.081 0 -0.004" rpy="-1.57 0 0"/>
-  </joint>
-  <link name="caster_back_link">
-    <collision>
-      <origin xyz="0 0.001 0" rpy="0 0 0"/>
-      <geometry>
-        <box size="0.030 0.009 0.020"/>
-      </geometry>
-    </collision>
-    <inertial>
-      <origin xyz="0 0 0" />
-      <mass value="0.005" />
+  <joint name="wheel_left_rear_joint" type="continuous">
+    <parent link="base_link"/>
+    <child link="wheel_left_rear_link"/>
+    <origin xyz="-0.060 0.078 0.023" rpy="-1.57 0 0"/>
+    <axis xyz="0 0 1"/>
+  </joint>
+  <link name="wheel_left_rear_link">
+    <visual>
+      <origin xyz="0 0 0" rpy="1.57 0 0"/>
+      <geometry>
+        <mesh filename="package://turtlebot3_description/meshes/wheels/left_tire.stl" scale="0.001 0.001 0.001"/>
+      </geometry>
+      <material name="dark"/>
+    </visual>
+    <collision>
+      <origin xyz="0 0 0" rpy="0 0 0"/>
+      <geometry>
+        <cylinder length="0.018" radius="0.033"/>
+      </geometry>
+    </collision>
+    <inertial>
+      <origin xyz="0 0 0" />
+      <mass value="2.8498940e-02" />
+      <inertia ixx="1.1175580e-05" ixy="0.0" ixz="0.0"
+               iyy="1.1192413e-05" iyz="0.0"
+               izz="2.0712558e-05" />
+    </inertial>
+  </link>
+  <joint name="wheel_right_rear_joint" type="continuous">
+    <parent link="base_link"/>
+    <child link="wheel_right_rear_link"/>
+    <origin xyz="-0.060 -0.078 0.023" rpy="-1.57 0 0"/>
+    <axis xyz="0 0 1"/>
+  </joint>
+  <link name="wheel_right_rear_link">
+    <visual>
+      <origin xyz="0 0 0" rpy="1.57 0 0"/>
+      <geometry>
+        <mesh filename="package://turtlebot3_description/meshes/wheels/right_tire.stl" scale="0.001 0.001 0.001"/>
+      </geometry>
+      <material name="dark"/>
+    </visual>
+    <collision>
+      <origin xyz="0 0 0" rpy="0 0 0"/>
+      <geometry>
+        <cylinder length="0.018" radius="0.033"/>
+      </geometry>
+    </collision>
+    <inertial>
+      <origin xyz="0 0 0" />
+      <mass value="2.8498940e-02" />
+      <inertia ixx="1.1175580e-05" ixy="0.0" ixz="0.0"
+               iyy="1.1192413e-05" iyz="0.0"
+               izz="2.0712558e-05" />
+    </inertial>
+  </link>
+  <joint name="imu_joint" type="fixed">
+    <parent link="base_link"/>
+    <child link="imu_link"/>
+    <origin xyz="-0.020 0 0.060" rpy="0 0 0"/>
+  </joint>
+  <link name="imu_link"/>
+  <joint name="scan_joint" type="fixed">
+    <parent link="base_link"/>
+    <child link="base_scan"/>
+    <origin xyz="0.035 0 0.085" rpy="0 0 0"/>
+  </joint>
+  <link name="base_scan">
+    <visual>
+      <origin xyz="0 0 0.0" rpy="0 0 0"/>
+      <geometry>
+        <mesh filename="package://turtlebot3_description/meshes/sensors/lds.stl" scale="0.001 0.001 0.001"/>
+      </geometry>
+      <material name="dark"/>
+    </visual>
+    <collision>
+      <origin xyz="0.015 0 -0.0065" rpy="0 0 0"/>
+      <geometry>
+        <cylinder length="0.0315" radius="0.055"/>
+      </geometry>
+    </collision>
+    <inertial>
+      <mass value="0.114" />
+      <origin xyz="0 0 0" />
       <inertia ixx="0.001" ixy="0.0" ixz="0.0"
                iyy="0.001" iyz="0.0"
@@ -778,36 +847,3 @@
     </inertial>
   </link>
-  <joint name="imu_joint" type="fixed">
-    <parent link="base_link"/>
-    <child link="imu_link"/>
-    <origin xyz="-0.020 0 0.060" rpy="0 0 0"/>
-  </joint>
-  <link name="imu_link"/>
-  <joint name="scan_joint" type="fixed">
-    <parent link="base_link"/>
-    <child link="base_scan"/>
-    <origin xyz="0.035 0 0.085" rpy="0 0 0"/>
-  </joint>
-  <link name="base_scan">
-    <visual>
-      <origin xyz="0 0 0.0" rpy="0 0 0"/>
-      <geometry>
-        <mesh filename="package://turtlebot3_description/meshes/sensors/lds.stl" scale="0.001 0.001 0.001"/>
-      </geometry>
-      <material name="dark"/>
-    </visual>
-    <collision>
-      <origin xyz="0.015 0 -0.0065" rpy="0 0 0"/>
-      <geometry>
-        <cylinder length="0.0315" radius="0.055"/>
-      </geometry>
-    </collision>
-    <inertial>
-      <mass value="0.114" />
-      <origin xyz="0 0 0" />
-      <inertia ixx="0.001" ixy="0.0" ixz="0.0"
-               iyy="0.001" iyz="0.0"
-               izz="0.001" />
-    </inertial>
-  </link>
 </robot>

Commit message: 四轮模型开源参考

File: src/turtlebot3/turtlebot3_description/urdf_next/turtlebot3_moguarder.gazebo.xacro (robot description, xacro)
@@ -79,36 +79,40 @@
   </gazebo>
   <gazebo reference="wheel_left_front_link">
-    <mu1>1.0</mu1>
-    <mu2>1.2</mu2>
-    <kp>500000.0</kp>
-    <kd>50.0</kd>
-    <minDepth>0.001</minDepth>
+    <mu1>1.00</mu1>
+    <mu2>0.35</mu2>
+    <kp>800000.0</kp>
+    <kd>8.0</kd>
+    <minDepth>0.001</minDepth>
+    <maxVel>0.1</maxVel>
     <fdir1>1 0 0</fdir1>
     <material>Gazebo/FlatBlack</material>
   </gazebo>
   <gazebo reference="wheel_right_front_link">
-    <mu1>1.0</mu1>
-    <mu2>1.2</mu2>
-    <kp>500000.0</kp>
-    <kd>50.0</kd>
-    <minDepth>0.001</minDepth>
+    <mu1>1.00</mu1>
+    <mu2>0.35</mu2>
+    <kp>800000.0</kp>
+    <kd>8.0</kd>
+    <minDepth>0.001</minDepth>
+    <maxVel>0.1</maxVel>
     <fdir1>1 0 0</fdir1>
     <material>Gazebo/FlatBlack</material>
   </gazebo>
   <gazebo reference="wheel_left_rear_link">
-    <mu1>1.0</mu1>
-    <mu2>1.2</mu2>
-    <kp>500000.0</kp>
-    <kd>50.0</kd>
-    <minDepth>0.001</minDepth>
+    <mu1>1.00</mu1>
+    <mu2>0.35</mu2>
+    <kp>800000.0</kp>
+    <kd>8.0</kd>
+    <minDepth>0.001</minDepth>
+    <maxVel>0.1</maxVel>
     <fdir1>1 0 0</fdir1>
     <material>Gazebo/FlatBlack</material>
   </gazebo>
   <gazebo reference="wheel_right_rear_link">
-    <mu1>1.0</mu1>
-    <mu2>1.2</mu2>
-    <kp>500000.0</kp>
-    <kd>50.0</kd>
-    <minDepth>0.001</minDepth>
+    <mu1>1.00</mu1>
+    <mu2>0.35</mu2>
+    <kp>800000.0</kp>
+    <kd>8.0</kd>
+    <minDepth>0.001</minDepth>
+    <maxVel>0.1</maxVel>
     <fdir1>1 0 0</fdir1>
     <material>Gazebo/FlatBlack</material>
@@ -132,7 +136,7 @@
       <leftRearJoint>wheel_left_rear_joint</leftRearJoint>
       <rightRearJoint>wheel_right_rear_joint</rightRearJoint>
-      <wheelSeparation>0.156</wheelSeparation>
-      <wheelDiameter>0.066</wheelDiameter>
-      <torque>12</torque>
+      <wheelSeparation>0.210</wheelSeparation>
+      <wheelDiameter>0.090</wheelDiameter>
+      <torque>18</torque>
       <broadcastTF>true</broadcastTF>
       <publishWheelTF>false</publishWheelTF>

File: src/turtlebot3/turtlebot3_description/urdf_next/turtlebot3_moguarder.urdf.xacro (robot description, xacro)
@@ -11,15 +11,15 @@
   <link name="base_link">
     <collision>
-      <origin xyz="-0.020 0 0.050" rpy="0 0 0"/>
-      <geometry>
-        <box size="0.135 0.130 0.105"/>
-      </geometry>
-    </collision>
-    <inertial>
-      <origin xyz="-0.010 0 0.035" rpy="0 0 0"/>
-      <mass value="8.2573504e-01"/>
-      <inertia ixx="1.8500000e-03" ixy="0.0" ixz="0.0"
-               iyy="1.9000000e-03" iyz="0.0"
-               izz="1.9500000e-03" />
+      <origin xyz="-0.010 0 0.060" rpy="0 0 0"/>
+      <geometry>
+        <box size="0.230 0.190 0.120"/>
+      </geometry>
+    </collision>
+    <inertial>
+      <origin xyz="-0.010 0 0.050" rpy="0 0 0"/>
+      <mass value="2.40"/>
+      <inertia ixx="1.60e-02" ixy="0.0" ixz="0.0"
+               iyy="2.20e-02" iyz="0.0"
+               izz="2.80e-02" />
     </inertial>
   </link>
@@ -54,5 +54,5 @@
     <parent link="base_link"/>
     <child link="front_shell_link"/>
-    <origin xyz="0.060 0 0.038" rpy="0 0 0"/>
+    <origin xyz="0.085 0 0.048" rpy="0 0 0"/>
   </joint>
   <link name="front_shell_link">
@@ -60,5 +60,5 @@
       <origin xyz="0 0 0" rpy="0 0 0"/>
       <geometry>
-        <box size="0.075 0.115 0.042"/>
+        <box size="0.090 0.165 0.045"/>
       </geometry>
       <material name="charcoal"/>
@@ -67,13 +67,13 @@
       <origin xyz="0 0 0" rpy="0 0 0"/>
       <geometry>
-        <box size="0.075 0.115 0.042"/>
-      </geometry>
-    </collision>
-    <inertial>
-      <origin xyz="0 0 0" />
-      <mass value="0.080" />
-      <inertia ixx="8.0e-05" ixy="0.0" ixz="0.0"
-               iyy="8.0e-05" iyz="0.0"
-               izz="1.0e-04" />
+        <box size="0.090 0.165 0.045"/>
+      </geometry>
+    </collision>
+    <inertial>
+      <origin xyz="0 0 0" />
+      <mass value="0.25" />
+      <inertia ixx="3.0e-04" ixy="0.0" ixz="0.0"
+               iyy="3.2e-04" iyz="0.0"
+               izz="4.0e-04" />
     </inertial>
   </link>
@@ -81,5 +81,5 @@
     <parent link="base_link"/>
     <child link="rear_module_link"/>
-    <origin xyz="-0.073 0 0.070" rpy="0 0 0"/>
+    <origin xyz="-0.090 0 0.078" rpy="0 0 0"/>
   </joint>
   <link name="rear_module_link">
@@ -87,5 +87,5 @@
       <origin xyz="0 0 0" rpy="0 0 0"/>
       <geometry>
-        <box size="0.050 0.105 0.060"/>
+        <box size="0.060 0.150 0.065"/>
       </geometry>
       <material name="matte_black"/>
@@ -94,13 +94,13 @@
       <origin xyz="0 0 0" rpy="0 0 0"/>
       <geometry>
-        <box size="0.050 0.105 0.060"/>
-      </geometry>
-    </collision>
-    <inertial>
-      <origin xyz="0 0 0" />
-      <mass value="0.090" />
-      <inertia ixx="7.0e-05" ixy="0.0" ixz="0.0"
-               iyy="7.5e-05" iyz="0.0"
-               izz="9.0e-05" />
+        <box size="0.060 0.150 0.065"/>
+      </geometry>
+    </collision>
+    <inertial>
+      <origin xyz="0 0 0" />
+      <mass value="0.40" />
+      <inertia ixx="6.0e-04" ixy="0.0" ixz="0.0"
+               iyy="6.5e-04" iyz="0.0"
+               izz="8.0e-04" />
     </inertial>
   </link>
@@ -108,5 +108,5 @@
     <parent link="base_link"/>
     <child link="front_bumper_link"/>
-    <origin xyz="0.105 0 0.030" rpy="0 0 0"/>
+    <origin xyz="0.130 0 0.043" rpy="0 0 0"/>
   </joint>
   <link name="front_bumper_link">
@@ -114,5 +114,5 @@
       <origin xyz="0 0 0" rpy="0 0 0"/>
       <geometry>
-        <box size="0.030 0.155 0.028"/>
+        <box size="0.035 0.215 0.030"/>
       </geometry>
       <material name="matte_black"/>
@@ -121,5 +121,5 @@
       <origin xyz="0 0 0" rpy="0 0 0"/>
       <geometry>
-        <box size="0.030 0.155 0.028"/>
+        <box size="0.035 0.215 0.030"/>
       </geometry>
     </collision>
@@ -705,5 +705,5 @@
     <parent link="base_link"/>
     <child link="wheel_left_front_link"/>
-    <origin xyz="0.060 0.078 0.023" rpy="-1.57 0 0"/>
+    <origin xyz="0.090 0.105 0.040" rpy="-1.57 0 0"/>
     <axis xyz="0 0 1"/>
   </joint>
@@ -719,13 +719,13 @@
       <origin xyz="0 0 0" rpy="0 0 0"/>
       <geometry>
-        <cylinder length="0.018" radius="0.033"/>
-      </geometry>
-    </collision>
-    <inertial>
-      <origin xyz="0 0 0" />
-      <mass value="2.8498940e-02" />
-      <inertia ixx="1.1175580e-05" ixy="0.0" ixz="0.0"
-               iyy="1.1192413e-05" iyz="0.0"
-               izz="2.0712558e-05" />
+        <cylinder length="0.028" radius="0.045"/>
+      </geometry>
+    </collision>
+    <inertial>
+      <origin xyz="0 0 0" />
+      <mass value="0.18" />
+      <inertia ixx="7.8e-05" ixy="0.0" ixz="0.0"
+               iyy="7.8e-05" iyz="0.0"
+               izz="1.45e-04" />
     </inertial>
   </link>
@@ -733,5 +733,5 @@
     <parent link="base_link"/>
     <child link="wheel_right_front_link"/>
-    <origin xyz="0.060 -0.078 0.023" rpy="-1.57 0 0"/>
+    <origin xyz="0.090 -0.105 0.040" rpy="-1.57 0 0"/>
     <axis xyz="0 0 1"/>
   </joint>
@@ -747,13 +747,13 @@
       <origin xyz="0 0 0" rpy="0 0 0"/>
       <geometry>
-        <cylinder length="0.018" radius="0.033"/>
-      </geometry>
-    </collision>
-    <inertial>
-      <origin xyz="0 0 0" />
-      <mass value="2.8498940e-02" />
-      <inertia ixx="1.1175580e-05" ixy="0.0" ixz="0.0"
-               iyy="1.1192413e-05" iyz="0.0"
-               izz="2.0712558e-05" />
+        <cylinder length="0.028" radius="0.045"/>
+      </geometry>
+    </collision>
+    <inertial>
+      <origin xyz="0 0 0" />
+      <mass value="0.18" />
+      <inertia ixx="7.8e-05" ixy="0.0" ixz="0.0"
+               iyy="7.8e-05" iyz="0.0"
+               izz="1.45e-04" />
     </inertial>
   </link>
@@ -761,5 +761,5 @@
     <parent link="base_link"/>
     <child link="wheel_left_rear_link"/>
-    <origin xyz="-0.060 0.078 0.023" rpy="-1.57 0 0"/>
+    <origin xyz="-0.090 0.105 0.040" rpy="-1.57 0 0"/>
     <axis xyz="0 0 1"/>
   </joint>
@@ -775,13 +775,13 @@
       <origin xyz="0 0 0" rpy="0 0 0"/>
       <geometry>
-        <cylinder length="0.018" radius="0.033"/>
-      </geometry>
-    </collision>
-    <inertial>
-      <origin xyz="0 0 0" />
-      <mass value="2.8498940e-02" />
-      <inertia ixx="1.1175580e-05" ixy="0.0" ixz="0.0"
-               iyy="1.1192413e-05" iyz="0.0"
-               izz="2.0712558e-05" />
+        <cylinder length="0.028" radius="0.045"/>
+      </geometry>
+    </collision>
+    <inertial>
+      <origin xyz="0 0 0" />
+      <mass value="0.18" />
+      <inertia ixx="7.8e-05" ixy="0.0" ixz="0.0"
+               iyy="7.8e-05" iyz="0.0"
+               izz="1.45e-04" />
     </inertial>
   </link>
@@ -789,5 +789,5 @@
     <parent link="base_link"/>
     <child link="wheel_right_rear_link"/>
-    <origin xyz="-0.060 -0.078 0.023" rpy="-1.57 0 0"/>
+    <origin xyz="-0.090 -0.105 0.040" rpy="-1.57 0 0"/>
     <axis xyz="0 0 1"/>
   </joint>
@@ -803,13 +803,13 @@
       <origin xyz="0 0 0" rpy="0 0 0"/>
       <geometry>
-        <cylinder length="0.018" radius="0.033"/>
-      </geometry>
-    </collision>
-    <inertial>
-      <origin xyz="0 0 0" />
-      <mass value="2.8498940e-02" />
-      <inertia ixx="1.1175580e-05" ixy="0.0" ixz="0.0"
-               iyy="1.1192413e-05" iyz="0.0"
-               izz="2.0712558e-05" />
+        <cylinder length="0.028" radius="0.045"/>
+      </geometry>
+    </collision>
+    <inertial>
+      <origin xyz="0 0 0" />
+      <mass value="0.18" />
+      <inertia ixx="7.8e-05" ixy="0.0" ixz="0.0"
+               iyy="7.8e-05" iyz="0.0"
+               izz="1.45e-04" />
     </inertial>
   </link>
