Commit message: 车基本模型最终版

File: src/turtlebot3/turtlebot3_description/urdf_next/turtlebot3_moguarder.gazebo.xacro (robot description, xacro)
@@ -27,10 +27,4 @@
     <material>Gazebo/FlatBlack</material>
   </gazebo>
-  <gazebo reference="lidar_guard_left_link">
-    <material>Gazebo/FlatBlack</material>
-  </gazebo>
-  <gazebo reference="lidar_guard_right_link">
-    <material>Gazebo/FlatBlack</material>
-  </gazebo>
   <gazebo reference="top_comm_module_link">
     <material>Gazebo/DarkGrey</material>
@@ -47,13 +41,4 @@
   <gazebo reference="right_yellow_trim_link">
     <material>Gazebo/Yellow</material>
-  </gazebo>
-  <gazebo reference="sensor_bridge_left_post_link">
-    <material>Gazebo/FlatBlack</material>
-  </gazebo>
-  <gazebo reference="sensor_bridge_right_post_link">
-    <material>Gazebo/FlatBlack</material>
-  </gazebo>
-  <gazebo reference="sensor_bridge_crossbar_link">
-    <material>Gazebo/FlatBlack</material>
   </gazebo>
   <gazebo reference="front_sensor_bezel_link">
@@ -136,5 +121,5 @@
       <leftRearJoint>wheel_left_rear_joint</leftRearJoint>
       <rightRearJoint>wheel_right_rear_joint</rightRearJoint>
-      <wheelSeparation>0.210</wheelSeparation>
+      <wheelSeparation>0.170</wheelSeparation>
       <wheelDiameter>0.090</wheelDiameter>
       <torque>18</torque>

File: src/turtlebot3/turtlebot3_description/urdf_next/turtlebot3_moguarder.urdf.xacro (robot description, xacro)
@@ -11,11 +11,11 @@
   <link name="base_link">
     <collision>
-      <origin xyz="-0.010 0 0.060" rpy="0 0 0"/>
-      <geometry>
-        <box size="0.230 0.190 0.120"/>
-      </geometry>
-    </collision>
-    <inertial>
-      <origin xyz="-0.010 0 0.050" rpy="0 0 0"/>
+      <origin xyz="-0.010 0 0.028" rpy="0 0 0"/>
+      <geometry>
+        <box size="0.220 0.155 0.055"/>
+      </geometry>
+    </collision>
+    <inertial>
+      <origin xyz="-0.010 0 0.048" rpy="0 0 0"/>
       <mass value="2.40"/>
       <inertia ixx="1.60e-02" ixy="0.0" ixz="0.0"
@@ -33,5 +33,5 @@
       <origin xyz="0 0 0" rpy="0 0 0"/>
       <geometry>
-        <box size="0.115 0.125 0.060"/>
+        <box size="0.110 0.105 0.060"/>
       </geometry>
       <material name="charcoal"/>
@@ -40,5 +40,5 @@
       <origin xyz="0 0 0" rpy="0 0 0"/>
       <geometry>
-        <box size="0.115 0.125 0.060"/>
+        <box size="0.110 0.105 0.060"/>
       </geometry>
     </collision>
@@ -54,5 +54,5 @@
     <parent link="base_link"/>
     <child link="front_shell_link"/>
-    <origin xyz="0.085 0 0.048" rpy="0 0 0"/>
+    <origin xyz="0.078 0 0.048" rpy="0 0 0"/>
   </joint>
   <link name="front_shell_link">
@@ -60,5 +60,5 @@
       <origin xyz="0 0 0" rpy="0 0 0"/>
       <geometry>
-        <box size="0.090 0.165 0.045"/>
+        <box size="0.080 0.125 0.045"/>
       </geometry>
       <material name="charcoal"/>
@@ -67,5 +67,5 @@
       <origin xyz="0 0 0" rpy="0 0 0"/>
       <geometry>
-        <box size="0.090 0.165 0.045"/>
+        <box size="0.080 0.125 0.045"/>
       </geometry>
     </collision>
@@ -87,5 +87,5 @@
       <origin xyz="0 0 0" rpy="0 0 0"/>
       <geometry>
-        <box size="0.060 0.150 0.065"/>
+        <box size="0.055 0.115 0.065"/>
       </geometry>
       <material name="matte_black"/>
@@ -94,5 +94,5 @@
       <origin xyz="0 0 0" rpy="0 0 0"/>
       <geometry>
-        <box size="0.060 0.150 0.065"/>
+        <box size="0.055 0.115 0.065"/>
       </geometry>
     </collision>
@@ -108,5 +108,5 @@
     <parent link="base_link"/>
     <child link="front_bumper_link"/>
-    <origin xyz="0.130 0 0.043" rpy="0 0 0"/>
+    <origin xyz="0.118 0 0.043" rpy="0 0 0"/>
   </joint>
   <link name="front_bumper_link">
@@ -114,5 +114,5 @@
       <origin xyz="0 0 0" rpy="0 0 0"/>
       <geometry>
-        <box size="0.035 0.215 0.030"/>
+        <box size="0.030 0.155 0.030"/>
       </geometry>
       <material name="matte_black"/>
@@ -121,5 +121,5 @@
       <origin xyz="0 0 0" rpy="0 0 0"/>
       <geometry>
-        <box size="0.035 0.215 0.030"/>
+        <box size="0.030 0.155 0.030"/>
       </geometry>
     </collision>
@@ -135,5 +135,5 @@
     <parent link="base_link"/>
     <child link="left_side_plate_link"/>
-    <origin xyz="-0.015 0.077 0.042" rpy="0 0 0"/>
+    <origin xyz="-0.015 0.060 0.042" rpy="0 0 0"/>
   </joint>
   <link name="left_side_plate_link">
@@ -141,5 +141,5 @@
       <origin xyz="0 0 0" rpy="0 0 0"/>
       <geometry>
-        <box size="0.145 0.014 0.040"/>
+        <box size="0.135 0.012 0.040"/>
       </geometry>
       <material name="matte_black"/>
@@ -148,5 +148,5 @@
       <origin xyz="0 0 0" rpy="0 0 0"/>
       <geometry>
-        <box size="0.145 0.014 0.040"/>
+        <box size="0.135 0.012 0.040"/>
       </geometry>
     </collision>
@@ -162,5 +162,5 @@
     <parent link="base_link"/>
     <child link="right_side_plate_link"/>
-    <origin xyz="-0.015 -0.077 0.042" rpy="0 0 0"/>
+    <origin xyz="-0.015 -0.060 0.042" rpy="0 0 0"/>
   </joint>
   <link name="right_side_plate_link">
@@ -168,5 +168,5 @@
       <origin xyz="0 0 0" rpy="0 0 0"/>
       <geometry>
-        <box size="0.145 0.014 0.040"/>
+        <box size="0.135 0.012 0.040"/>
       </geometry>
       <material name="dark"/>
@@ -175,5 +175,5 @@
       <origin xyz="0 0 0" rpy="0 0 0"/>
       <geometry>
-        <box size="0.145 0.014 0.040"/>
+        <box size="0.135 0.012 0.040"/>
       </geometry>
     </collision>
@@ -189,5 +189,5 @@
     <parent link="base_link"/>
     <child link="lidar_mount_link"/>
-    <origin xyz="0.035 0 0.052" rpy="0 0 0"/>
+    <origin xyz="0.060 0 0.075" rpy="0 0 0"/>
   </joint>
   <link name="lidar_mount_link">
@@ -195,5 +195,5 @@
       <origin xyz="0 0 0" rpy="0 0 0"/>
       <geometry>
-        <box size="0.060 0.072 0.014"/>
+        <box size="0.048 0.060 0.014"/>
       </geometry>
       <material name="dark"/>
@@ -202,5 +202,5 @@
       <origin xyz="0 0 0" rpy="0 0 0"/>
       <geometry>
-        <box size="0.060 0.072 0.014"/>
+        <box size="0.048 0.060 0.014"/>
       </geometry>
     </collision>
@@ -213,58 +213,4 @@
     </inertial>
   </link>
-  <joint name="lidar_guard_left_joint" type="fixed">
-    <parent link="base_link"/>
-    <child link="lidar_guard_left_link"/>
-    <origin xyz="0.035 0.044 0.086" rpy="0 0 0"/>
-  </joint>
-  <link name="lidar_guard_left_link">
-    <visual>
-      <origin xyz="0 0 0" rpy="0 0 0"/>
-      <geometry>
-        <box size="0.070 0.010 0.050"/>
-      </geometry>
-      <material name="matte_black"/>
-    </visual>
-    <collision>
-      <origin xyz="0 0 0" rpy="0 0 0"/>
-      <geometry>
-        <box size="0.070 0.010 0.050"/>
-      </geometry>
-    </collision>
-    <inertial>
-      <origin xyz="0 0 0" />
-      <mass value="0.018" />
-      <inertia ixx="8.0e-06" ixy="0.0" ixz="0.0"
-               iyy="8.0e-06" iyz="0.0"
-               izz="9.0e-06" />
-    </inertial>
-  </link>
-  <joint name="lidar_guard_right_joint" type="fixed">
-    <parent link="base_link"/>
-    <child link="lidar_guard_right_link"/>
-    <origin xyz="0.035 -0.044 0.086" rpy="0 0 0"/>
-  </joint>
-  <link name="lidar_guard_right_link">
-    <visual>
-      <origin xyz="0 0 0" rpy="0 0 0"/>
-      <geometry>
-        <box size="0.070 0.010 0.050"/>
-      </geometry>
-      <material name="matte_black"/>
-    </visual>
-    <collision>
-      <origin xyz="0 0 0" rpy="0 0 0"/>
-      <geometry>
-        <box size="0.070 0.010 0.050"/>
-      </geometry>
-    </collision>
-    <inertial>
-      <origin xyz="0 0 0" />
-      <mass value="0.018" />
-      <inertia ixx="8.0e-06" ixy="0.0" ixz="0.0"
-               iyy="8.0e-06" iyz="0.0"
-               izz="9.0e-06" />
-    </inertial>
-  </link>
   <joint name="top_comm_module_joint" type="fixed">
     <parent link="base_link"/>
@@ -297,5 +243,5 @@
     <parent link="base_link"/>
     <child link="left_range_link"/>
-    <origin xyz="0.020 0.090 0.055" rpy="0 0 1.5708"/>
+    <origin xyz="0.020 0.074 0.055" rpy="0 0 1.5708"/>
   </joint>
   <link name="left_range_link">
@@ -324,5 +270,5 @@
     <parent link="base_link"/>
     <child link="right_range_link"/>
-    <origin xyz="0.020 -0.090 0.055" rpy="0 0 -1.5708"/>
+    <origin xyz="0.020 -0.074 0.055" rpy="0 0 -1.5708"/>
   </joint>
   <link name="right_range_link">
@@ -357,5 +303,5 @@
       <origin xyz="0 0 0" rpy="0 0 0"/>
       <geometry>
-        <box size="0.165 0.135 0.010"/>
+        <box size="0.155 0.110 0.010"/>
       </geometry>
       <material name="matte_black"/>
@@ -364,5 +310,5 @@
       <origin xyz="0 0 0" rpy="0 0 0"/>
       <geometry>
-        <box size="0.165 0.135 0.010"/>
+        <box size="0.155 0.110 0.010"/>
       </geometry>
     </collision>
@@ -384,5 +330,5 @@
       <origin xyz="0 0 0" rpy="0 0 0"/>
       <geometry>
-        <box size="0.010 0.145 0.012"/>
+        <box size="0.010 0.112 0.012"/>
       </geometry>
       <material name="safety_yellow"/>
@@ -391,5 +337,5 @@
       <origin xyz="0 0 0" rpy="0 0 0"/>
       <geometry>
-        <box size="0.010 0.145 0.012"/>
+        <box size="0.010 0.112 0.012"/>
       </geometry>
     </collision>
@@ -405,5 +351,5 @@
     <parent link="base_link"/>
     <child link="left_yellow_trim_link"/>
-    <origin xyz="-0.015 0.085 0.061" rpy="0 0 0"/>
+    <origin xyz="-0.015 0.068 0.061" rpy="0 0 0"/>
   </joint>
   <link name="left_yellow_trim_link">
@@ -411,5 +357,5 @@
       <origin xyz="0 0 0" rpy="0 0 0"/>
       <geometry>
-        <box size="0.140 0.008 0.012"/>
+        <box size="0.130 0.007 0.012"/>
       </geometry>
       <material name="safety_yellow"/>
@@ -418,5 +364,5 @@
       <origin xyz="0 0 0" rpy="0 0 0"/>
       <geometry>
-        <box size="0.140 0.008 0.012"/>
+        <box size="0.130 0.007 0.012"/>
       </geometry>
     </collision>
@@ -432,5 +378,5 @@
     <parent link="base_link"/>
     <child link="right_yellow_trim_link"/>
-    <origin xyz="-0.015 -0.085 0.061" rpy="0 0 0"/>
+    <origin xyz="-0.015 -0.068 0.061" rpy="0 0 0"/>
   </joint>
   <link name="right_yellow_trim_link">
@@ -438,5 +384,5 @@
       <origin xyz="0 0 0" rpy="0 0 0"/>
       <geometry>
-        <box size="0.140 0.008 0.012"/>
+        <box size="0.130 0.007 0.012"/>
       </geometry>
       <material name="safety_yellow"/>
@@ -445,5 +391,5 @@
       <origin xyz="0 0 0" rpy="0 0 0"/>
       <geometry>
-        <box size="0.140 0.008 0.012"/>
+        <box size="0.130 0.007 0.012"/>
       </geometry>
     </collision>
@@ -456,85 +402,4 @@
     </inertial>
   </link>
-  <joint name="sensor_bridge_left_post_joint" type="fixed">
-    <parent link="base_link"/>
-    <child link="sensor_bridge_left_post_link"/>
-    <origin xyz="0.035 0.048 0.107" rpy="0 0 0"/>
-  </joint>
-  <link name="sensor_bridge_left_post_link">
-    <visual>
-      <origin xyz="0 0 0" rpy="0 0 0"/>
-      <geometry>
-        <box size="0.010 0.010 0.052"/>
-      </geometry>
-      <material name="matte_black"/>
-    </visual>
-    <collision>
-      <origin xyz="0 0 0" rpy="0 0 0"/>
-      <geometry>
-        <box size="0.010 0.010 0.052"/>
-      </geometry>
-    </collision>
-    <inertial>
-      <origin xyz="0 0 0" />
-      <mass value="0.012" />
-      <inertia ixx="5.0e-06" ixy="0.0" ixz="0.0"
-               iyy="5.0e-06" iyz="0.0"
-               izz="5.0e-06" />
-    </inertial>
-  </link>
-  <joint name="sensor_bridge_right_post_joint" type="fixed">
-    <parent link="base_link"/>
-    <child link="sensor_bridge_right_post_link"/>
-    <origin xyz="0.035 -0.048 0.107" rpy="0 0 0"/>
-  </joint>
-  <link name="sensor_bridge_right_post_link">
-    <visual>
-      <origin xyz="0 0 0" rpy="0 0 0"/>
-      <geometry>
-        <box size="0.010 0.010 0.052"/>
-      </geometry>
-      <material name="matte_black"/>
-    </visual>
-    <collision>
-      <origin xyz="0 0 0" rpy="0 0 0"/>
-      <geometry>
-        <box size="0.010 0.010 0.052"/>
-      </geometry>
-    </collision>
-    <inertial>
-      <origin xyz="0 0 0" />
-      <mass value="0.012" />
-      <inertia ixx="5.0e-06" ixy="0.0" ixz="0.0"
-               iyy="5.0e-06" iyz="0.0"
-               izz="5.0e-06" />
-    </inertial>
-  </link>
-  <joint name="sensor_bridge_crossbar_joint" type="fixed">
-    <parent link="base_link"/>
-    <child link="sensor_bridge_crossbar_link"/>
-    <origin xyz="0.035 0 0.128" rpy="0 0 0"/>
-  </joint>
-  <link name="sensor_bridge_crossbar_link">
-    <visual>
-      <origin xyz="0 0 0" rpy="0 0 0"/>
-      <geometry>
-        <box size="0.070 0.112 0.010"/>
-      </geometry>
-      <material name="matte_black"/>
-    </visual>
-    <collision>
-      <origin xyz="0 0 0" rpy="0 0 0"/>
-      <geometry>
-        <box size="0.070 0.112 0.010"/>
-      </geometry>
-    </collision>
-    <inertial>
-      <origin xyz="0 0 0" />
-      <mass value="0.020" />
-      <inertia ixx="7.0e-06" ixy="0.0" ixz="0.0"
-               iyy="7.0e-06" iyz="0.0"
-               izz="9.0e-06" />
-    </inertial>
-  </link>
   <joint name="front_sensor_bezel_joint" type="fixed">
     <parent link="base_link"/>
@@ -567,5 +432,5 @@
     <parent link="base_link"/>
     <child link="left_sensor_bezel_link"/>
-    <origin xyz="0.020 0.101 0.055" rpy="0 0 0"/>
+    <origin xyz="0.020 0.083 0.055" rpy="0 0 0"/>
   </joint>
   <link name="left_sensor_bezel_link">
@@ -594,5 +459,5 @@
     <parent link="base_link"/>
     <child link="right_sensor_bezel_link"/>
-    <origin xyz="0.020 -0.101 0.055" rpy="0 0 0"/>
+    <origin xyz="0.020 -0.083 0.055" rpy="0 0 0"/>
   </joint>
   <link name="right_sensor_bezel_link">
@@ -621,5 +486,5 @@
     <parent link="base_link"/>
     <child link="deck_fastener_fl_link"/>
-    <origin xyz="0.045 0.048 0.095" rpy="0 0 0"/>
+    <origin xyz="0.045 0.040 0.095" rpy="0 0 0"/>
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
Commit message: 雷达270调整，摄像头添加

File: src/turtlebot3/turtlebot3_description/urdf_next/turtlebot3_moguarder.gazebo.xacro (robot description, xacro)
@@ -26,4 +26,10 @@
   <gazebo reference="lidar_mount_link">
     <material>Gazebo/FlatBlack</material>
+  </gazebo>
+  <gazebo reference="camera_mount_link">
+    <material>Gazebo/FlatBlack</material>
+  </gazebo>
+  <gazebo reference="camera_link">
+    <material>Gazebo/Black</material>
   </gazebo>
   <gazebo reference="top_comm_module_link">
@@ -169,6 +175,6 @@
             <samples>720</samples>
             <resolution>1</resolution>
-            <min_angle>0.0</min_angle>
-            <max_angle>6.28319</max_angle>
+            <min_angle>-2.35619</min_angle>
+            <max_angle>2.35619</max_angle>
           </horizontal>
         </scan>
@@ -187,4 +193,37 @@
         <topicName>scan</topicName>
         <frameName>base_scan</frameName>
+      </plugin>
+    </sensor>
+  </gazebo>
+  <gazebo reference="camera_link">
+    <sensor type="camera" name="moguarder_front_camera">
+      <pose>0 0 0 0 0 0</pose>
+      <visualize>true</visualize>
+      <update_rate>30</update_rate>
+      <camera>
+        <horizontal_fov>1.22173</horizontal_fov>
+        <image>
+          <width>640</width>
+          <height>480</height>
+          <format>R8G8B8</format>
+        </image>
+        <clip>
+          <near>0.03</near>
+          <far>20.0</far>
+        </clip>
+      </camera>
+      <plugin name="moguarder_front_camera_controller" filename="libgazebo_ros_camera.so">
+        <alwaysOn>true</alwaysOn>
+        <updateRate>30</updateRate>
+        <cameraName>camera/rgb</cameraName>
+        <imageTopicName>/camera/rgb/image_raw</imageTopicName>
+        <cameraInfoTopicName>/camera/rgb/camera_info</cameraInfoTopicName>
+        <frameName>camera_link</frameName>
+        <hackBaseline>0.0</hackBaseline>
+        <distortionK1>0.0</distortionK1>
+        <distortionK2>0.0</distortionK2>
+        <distortionK3>0.0</distortionK3>
+        <distortionT1>0.0</distortionT1>
+        <distortionT2>0.0</distortionT2>
       </plugin>
     </sensor>

File: src/turtlebot3/turtlebot3_description/urdf_next/turtlebot3_moguarder.urdf.xacro (robot description, xacro)
@@ -213,4 +213,65 @@
     </inertial>
   </link>
+  <joint name="camera_mount_joint" type="fixed">
+    <parent link="base_link"/>
+    <child link="camera_mount_link"/>
+    <origin xyz="0.080 0 0.105" rpy="0 0 0"/>
+  </joint>
+  <link name="camera_mount_link">
+    <visual>
+      <origin xyz="0 0 0" rpy="0 0 0"/>
+      <geometry>
+        <box size="0.052 0.050 0.014"/>
+      </geometry>
+      <material name="matte_black"/>
+    </visual>
+    <collision>
+      <origin xyz="0 0 0" rpy="0 0 0"/>
+      <geometry>
+        <box size="0.052 0.050 0.014"/>
+      </geometry>
+    </collision>
+    <inertial>
+      <origin xyz="0 0 0" />
+      <mass value="0.025" />
+      <inertia ixx="8.0e-06" ixy="0.0" ixz="0.0"
+               iyy="8.0e-06" iyz="0.0"
+               izz="1.0e-05" />
+    </inertial>
+  </link>
+  <joint name="camera_joint" type="fixed">
+    <parent link="camera_mount_link"/>
+    <child link="camera_link"/>
+    <origin xyz="0.018 0 0.020" rpy="0 0 0"/>
+  </joint>
+  <link name="camera_link">
+    <visual>
+      <origin xyz="0 0 0" rpy="0 0 0"/>
+      <geometry>
+        <box size="0.030 0.036 0.024"/>
+      </geometry>
+      <material name="dark"/>
+    </visual>
+    <visual>
+      <origin xyz="0.016 0 0" rpy="0 1.5708 0"/>
+      <geometry>
+        <cylinder length="0.006" radius="0.010"/>
+      </geometry>
+      <material name="sensor_glass"/>
+    </visual>
+    <collision>
+      <origin xyz="0 0 0" rpy="0 0 0"/>
+      <geometry>
+        <box size="0.030 0.036 0.024"/>
+      </geometry>
+    </collision>
+    <inertial>
+      <origin xyz="0 0 0" />
+      <mass value="0.035" />
+      <inertia ixx="1.2e-05" ixy="0.0" ixz="0.0"
+               iyy="1.2e-05" iyz="0.0"
+               izz="1.4e-05" />
+    </inertial>
+  </link>
   <joint name="top_comm_module_joint" type="fixed">
     <parent link="base_link"/>
